File: Oszi/KiCad/OsziFrontEnd/muC.kicad_sch (KiCad schematic)
At the start: 1 part, among them U3 NUCLEO-L432KC

Commit message: startet coding and configure .ios
Parts:
- U3: footprint L432KC:MODULE_NUCLEO-L432KC -> My_Connectors:NUCLEO-L432KC_Module
Connections:
- net ADC_CH1_10V: now also U3.CN4_11 (PA1); no longer U3.CN3_9 (PB1)
- net ADC_CH1_1V: now also U3.CN4_12 (PA0); no longer U3.CN3_6 (PB0)
- net ADC_CH2_10V: now also U3.CN4_10 (PA3); no longer U3.CN4_11 (PA1)
- net ADC_CH2_36V: now also U3.CN4_5 (PA2); no longer U3.CN4_12 (PA0)
- net 5V: no longer names the net of U3.CN4_4 (+5V)
- no-connect marks 22 -> 23
Other:
- note added: "DC-Pin"
- note added: "Display reset"
- note added: "Spannungsregler kann bis zu 500mA"
- note added: "W5500 reset for reset 10k pull up"
- note removed: "Spannungsregler kann bis zu 300mA"
Changed lines of the file:
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@@
 	(generator_version "9.0")
 	(paper "A4")
-	(text "Spannungsregler kann bis zu 300mA\n"
+	(text "Display reset\n"
+		(exclude_from_sim no)
+		(at 249.682 68.834 0)
+		(effects
+			(font
+				(size 1.27 1.27)
+				(thickness 0.254)
+				(bold yes)
+			)
+		)
+	)
+	(text "DC-Pin"
+		(exclude_from_sim no)
+		(at 248.158 61.214 0)
+		(effects
+			(font
+				(size 1.27 1.27)
+				(thickness 0.254)
+				(bold yes)
+			)
+		)
+	)
+	(text "W5500 reset\n\nfor reset 10k pull up\n"
+		(exclude_from_sim no)
+		(at 249.936 75.946 0)
+		(effects
+			(font
+				(size 1.27 1.27)
+				(thickness 0.254)
+				(bold yes)
+			)
+		)
+	)
+	(text "Spannungsregler kann bis zu 500mA\n"
 		(exclude_from_sim no)
 		(at 255.778 120.396 0)
@@
 	)
 	(no_connect
-		(at 212.09 147.32)
-	)
-	(no_connect
 		(at 212.09 63.5)
 	)
 	(no_connect
+		(at 242.57 124.46)
+	)
+	(no_connect
 		(at 242.57 144.78)
 	)
@@
 	)
 	(no_connect
+		(at 242.57 63.5)
+	)
+	(no_connect
+		(at 242.57 60.96)
+	)
+	(no_connect
 		(at 212.09 60.96)
 	)
@@
 	(no_connect
 		(at 242.57 132.08)
-	)
-	(no_connect
-		(at 212.09 149.86)
 	)
 	(no_connect
@@
 	(wire
 		(pts
-			(xy 242.57 60.96) (xy 247.65 60.96)
+			(xy 242.57 127) (xy 245.11 127)
 		)
 		(stroke
@@
 	(wire
 		(pts
-			(xy 242.57 127) (xy 245.11 127)
+			(xy 242.57 154.94) (xy 242.57 157.48)
 		)
 		(stroke
@@
 	(wire
 		(pts
-			(xy 242.57 154.94) (xy 242.57 157.48)
+			(xy 208.28 144.78) (xy 212.09 144.78)
 		)
 		(stroke
@@
 	(wire
 		(pts
-			(xy 208.28 144.78) (xy 212.09 144.78)
+			(xy 208.28 142.24) (xy 212.09 142.24)
 		)
 		(stroke
@@
 	(wire
 		(pts
-			(xy 208.28 142.24) (xy 212.09 142.24)
+			(xy 208.28 149.86) (xy 212.09 149.86)
 		)
 		(stroke
@@
 	(wire
 		(pts
-			(xy 242.57 63.5) (xy 247.65 63.5)
+			(xy 208.28 147.32) (xy 212.09 147.32)
 		)
 		(stroke
@@
 	(hierarchical_label "ADC_CH2_36V"
 		(shape input)
-		(at 208.28 142.24 180)
+		(at 208.28 147.32 180)
 		(effects
 			(font
@@
 			)
 			(justify right)
-		)
-	)
-	(hierarchical_label "5V"
-		(shape input)
-		(at 242.57 124.46 0)
-		(effects
-			(font
-				(size 1.27 1.27)
-				(thickness 0.254)
-				(bold yes)
-			)
-			(justify left)
 		)
 	)
@@
 	(hierarchical_label "ADC_CH2_10V"
 		(shape input)
-		(at 208.28 144.78 180)
+		(at 208.28 149.86 180)
 		(effects
 			(font
@@
 	(hierarchical_label "ADC_CH1_10V"
 		(shape input)
-		(at 247.65 63.5 0)
-		(effects
-			(font
-				(size 1.27 1.27)
-				(thickness 0.254)
-				(bold yes)
-			)
-			(justify left)
+		(at 208.28 144.78 180)
+		(effects
+			(font
+				(size 1.27 1.27)
+				(thickness 0.254)
+				(bold yes)
+			)
+			(justify right)
 		)
 	)
 	(hierarchical_label "ADC_CH1_1V"
 		(shape input)
-		(at 247.65 60.96 0)
-		(effects
-			(font
-				(size 1.27 1.27)
-				(thickness 0.254)
-				(bold yes)
-			)
-			(justify left)
+		(at 208.28 142.24 180)
+		(effects
+			(font
+				(size 1.27 1.27)
+				(thickness 0.254)
+				(bold yes)
+			)
+			(justify right)
 		)
 	)
@@
 			)
 		)
-		(property "Footprint" "L432KC:MODULE_NUCLEO-L432KC"
+		(property "Footprint" "My_Connectors:NUCLEO-L432KC_Module"
 			(at 227.33 139.7 0)
 			(effects
@@
 			)
 		)
-		(property "Footprint" "L432KC:MODULE_NUCLEO-L432KC"
+		(property "Footprint" "My_Connectors:NUCLEO-L432KC_Module"
 			(at 227.33 68.58 0)
 			(effects
