File: Oszi/KiCad/OsziFrontEnd/muC.kicad_sch (KiCad schematic)
At the start: 1 part, among them U3 NUCLEO-L432KC

Commit message: finished layout
Parts:
- added RV1: R_Potentiometer, Potentiometer_SMD:Potentiometer_ACP_CA6-VSMD_Vertical, symbol Device:R_Potentiometer
- added SW1, SW2, SW3: SW_Push, Button_Switch_SMD:SW_SPST_PTS645Sx43SMTR92, symbol Switch:SW_Push
Connections:
- net 3V3: now also RV1.3, SW1.1, SW2.1, SW3.2
- net MOSI: now reaches U3.CN4_6 (PA7)
- net MISO: now reaches U3.CN4_7 (PA6)
- net SCK: now reaches U3.CN4_8 (PA5)
- net at U3.CN3_1 (PA9): now also RV1.2
- net EINT: now reaches U3.CN3_12 (PA8)
- net at U3.CN3_13 (PA11): now also SW2.2
- net at U3.CN3_14 (PB5): now also SW3.1
- net DRs: now reaches U3.CN3_15 (PB4)
- net at U3.CN3_2 (PA10): now also SW1.2
- net DCS: now reaches U3.CN3_6 (PB0)
- net ERs: now reaches U3.CN3_7 (PB7)
- net ECS: now reaches U3.CN3_8 (PB6)
- net DD/C: now reaches U3.CN3_9 (PB1)
- new net GND: RV1.1
- no-connect marks 23 -> 9
Other:
- note added: "PB7, 6, PA8"
- note removed: "DC-Pin"
- note removed: "Display reset"
- note removed: "W5500 reset for reset 10k pull up"
- moved on the sheet: U3B
