File: Oszi/KiCad/OsziFrontEnd/powerSupplie.kicad_sch (KiCad schematic)
At the start: 3 parts, among them J5 USB_C_Receptacle_PowerOnly_6P

Commit message: startet coding and configure .ios
Parts:
- added C2: 10u, Capacitor_SMD:C_0603_1608Metric_Pad1.08x0.95mm_HandSolder, symbol Device:C
- added C3: 22u, Capacitor_SMD:C_0603_1608Metric_Pad1.08x0.95mm_HandSolder, symbol Device:C
- added L1: 2.2u, Inductor_SMD:L_0603_1608Metric, symbol Device:L
- added R21: 330k, Resistor_SMD:R_0603_1608Metric, symbol Device:R
- added R22: 100k, Resistor_SMD:R_0603_1608Metric, symbol Device:R
- added U4: TPS62160DGK, Package_SO:MSOP-8_3x3mm_P0.65mm, symbol Regulator_Switching:TPS62160DGK
Connections:
- net GND: now also C2.2, R22.2, U4.1 (PGND), U4.4 (AGND)
- net USB-cOut: now also C2.1, U4.2 (VIN), U4.3 (EN)
- new net: L1.1, U4.7 (SW)
- new net: C3.2, R22.1, U4.5 (FB)
- new net: R21.2, U4.8 (PG)
- new net 3V3: C3.1, L1.2, R21.1, U4.6 (VOS)
Other:
- note added: "LQM2HPN2R2MJHL"
- moved on the sheet: J5, R19, R20
