File: Oszi/KiCad/OsziFrontEnd/AnalogesFrontEnd.kicad_sch (KiCad schematic)
At the start: 25 parts, among them J1 Conn_Coaxial, J2 Conn_Coaxial, J3 Conn_01x03_Pin, J4 Conn_01x03_Pin, U1 MCP6002-xP, U2 MCP6002-xP

Commit message: startet coding and configure .ios
Changed lines of the file:
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@@
 	)
 	(rectangle
-		(start 158.75 35.56)
+		(start 158.75 33.02)
 		(end 241.3 140.97)
 		(stroke

Commit message: finished layout
Connections:
- net Vin-10;10CH1: no longer R1.1
- net Vin-1;1CH1: now also R1.1
Changed lines of the file:
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@@
+		)
+	)
+	(hierarchical_label "Vin-1;1CH1"
+		(shape input)
+		(at 209.55 50.8 90)
+		(effects
+			(font
+				(size 1.27 1.27)
+				(thickness 0.254)
+				(bold yes)
+			)
+			(justify left)
 		)
 	)
@@
 		(effects
 			(font
-				(size 1.27 1.27)
-				(thickness 0.254)
-				(bold yes)
-			)
-			(justify left)
-		)
-	)
-	(hierarchical_label "Vin-10;10CH1"
-		(shape input)
-		(at 209.55 50.8 90)
-		(effects
-			(font
