File: Oszi/KiCad/OsziFrontEnd/_autosave-OsziFrontEnd.kicad_pcb (KiCad board)
At the start: 2 copper layers, 91.9 x 85.4 mm, 42 parts, among them J1 Conn_Coaxial, J2 Conn_Coaxial, J3 Conn_01x03_Pin, J4 Conn_01x03_Pin, J5 USB_C_Receptacle_PowerOnly_6P, U1 MCP6002-xP, U2 MCP6002-xP, U3 NUCLEO-L432KC, U4 TPS62160DGK, U6 CR2013-MI2120

Commit message: added CubeIDE project
Parts:
- moved R9 6.50 mm to (103.2, 83.8)
- moved J4 6.09 mm to (94.1, 83.6)
- moved R17 6.09 mm to (103.9, 82.2)
- moved R8 6.09 mm to (97.2, 83.2)
- moved R10 6.09 mm to (101.5, 86.0)
- moved R11 6.09 mm to (97.3, 86.2)
- moved R7 6.09 mm to (100.0, 82.9)
- moved CH Select 6.02 mm to (145.8, 75.7)
- moved Mode Select 5.97 mm to (145.6, 84.9)
- moved Run / Stop 5.76 mm to (145.8, 67.0)
- moved Trimm 5.73 mm to (146.4, 94.5)
- moved U3 5.64 mm to (138.3, 97.7)
- moved C2 1.76 mm to (88.6, 69.0)
- moved C4 1.42 mm to (83.1, 29.8)
- moved U6 1.40 mm to (85.9, 28.5)
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Routing:
- net 3V3: track 237.8 -> 247.4 mm
- net /Display/DD/C: track 83.5 -> 75.7 mm
- net /Display/DSCK: track 78.4 -> 72.0 mm
- net /AnalogesFrontEnd/ADC_CH1_1V: track 26.2 -> 20.5 mm
- net /AnalogesFrontEnd/ADC_CH1_10V: track 16.7 -> 11.1 mm
- net /AnalogesFrontEnd/ADC_CH2_36V: track 27.8 -> 22.1 mm
- net /Display/DMOSI: track 76.7 -> 71.8 mm
- net /Display/DRs: track 77.8 -> 72.9 mm
- net /Display/DMISO: track 71.1 -> 66.4 mm
- net Net-(U2A-+): track 2.63 -> 7.32 mm
- net /AnalogesFrontEnd/ADC_CH2_10V: track 19.3 -> 15.0 mm
- net /AnalogesFrontEnd/CoaxCH2: track 10.8 -> 6.88 mm
- net /Display/DCS: track 92.7 -> 88.9 mm
- net /AnalogesFrontEnd/Vout-10;10CH2: track 17.9 -> 21.7 mm
- net GNDD: track 17.3 -> 19.7 mm, vias 0 -> 1
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Other:
- board size 91.9 x 85.4 mm -> 75.3 x 85.4 mm
