File: Oszi/KiCad/OsziFrontEnd/Display.kicad_sch (KiCad schematic)
At the start: 0 parts

Commit message: finished layout
Parts:
- added C4: 12p, symbol Device:C
- added R23: 10k, symbol Device:R
- added U6: CR2013-MI2120, Display:CR2013-MI2120, symbol Driver_Display:CR2013-MI2120
Connections:
- new net 3V3: C4.2, R23.2, U6.1 (VCC), U6.8 (LED)
- new net DCS: U6.3 (~{CS})
- new net DD/C: U6.5 (D/~{C})
- new net DMISO: U6.9 (MISO)
- new net DMOSI: U6.6 (MOSI)
- new net DRs: R23.1, U6.4 (RESET)
- new net DSCK: U6.7 (SCK)
- new net GND: C4.1, U6.2 (GND)
- no-connect marks 0 -> 5

Commit message: finished layout
Parts:
- C4: footprint (none) -> Capacitor_SMD:C_0603_1608Metric
- R23: footprint (none) -> Resistor_SMD:R_0603_1608Metric
Changed lines of the file:
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@@
 			)
 		)
-		(property "Footprint" ""
+		(property "Footprint" "Capacitor_SMD:C_0603_1608Metric"
 			(at 125.73 77.5208 0)
 			(effects
@@
 			)
 		)
-		(property "Footprint" ""
+		(property "Footprint" "Resistor_SMD:R_0603_1608Metric"
 			(at 153.162 109.474 90)
 			(effects

Commit message: jetzt git
Parts:
- added J6: Conn_01x14_Socket, Connector_PinSocket_2.54mm:PinSocket_1x14_P2.54mm_Vertical, symbol Connector:Conn_01x14_Socket
- added J7: Conn_01x04_Socket, Connector_PinSocket_2.54mm:PinSocket_1x04_P2.54mm_Vertical, symbol Connector:Conn_01x04_Socket
Connections:
- net 3V3: now also J6.1 (Pin_1), J6.8 (Pin_8)
- net DCS: now also J6.3 (Pin_3)
- net DD/C: now also J6.5 (Pin_5)
- net DMISO: now also J6.9 (Pin_9)
- net DMOSI: now also J6.6 (Pin_6)
- net DRs: now also J6.4 (Pin_4)
- net DSCK: now also J6.7 (Pin_7)
- net GND: now also J6.2 (Pin_2)
- no-connect marks 5 -> 14
